Commit message: working simulation

File: docker/shelfino_gazebo/models/shelfino/model.urdf (robot description, URDF)
Before this commit: robot shelfino, 4 links, 3 joints
Links:
- link base_laser: geometry collision cylinder length=0.04 radius=0.023; visual mesh filename=package://shelfino_gazebo/models/lidar2d/meshes/hokuyo.dae
- link base_link: geometry collision box size=.5 .5 .45; visual box size=.5 .5 .4

Commit message: simulator update

File: docker/shelfino_gazebo/models/shelfino/model.urdf (robot description, URDF)
Before this commit: robot shelfino, 4 links, 3 joints
Links:
- link base_laser: geometry collision cylinder length=0.04 radius=0.023; visual mesh filename=model://lidar2d/meshes/hokuyo.dae
Joints:
- joint lidar2d_joint: origin xyz=0 0 0.45 rpy=0 0 0 -> xyz=0 0 0.51 rpy=0 0 0

Commit message: reverted to using both sdf and urdf for the robot description

File: docker/shelfino_gazebo/models/shelfino/model.urdf (robot description, URDF)
Before this commit: robot shelfino, 4 links, 3 joints
Links:
- link base_laser: geometry collision cylinder length=0.04 radius=0.023; visual mesh filename=package://shelfino_gazebo/models/lidar2d/meshes/hokuyo.dae
Joints:
- joint lidar2d_joint: origin xyz=0 0 0.51 rpy=0 0 0 -> xyz=0 0 0.45 rpy=0 0 0
