Commit message: Changed URDF to a XACRO to specify the robot_name and be able to use multiple robots

File: shelfino_description/models/shelfino/model.xacro (robot description, xacro)
@@ -16,5 +16,5 @@
                                                       BODY OF SHELFINO
 -->
-  <link name='base_link'>
+  <link name='shelfino2/base_link'>
     <visual name='body_visual'>
       <origin xyz='0 0 .25'/>
@@ -49,6 +49,6 @@
 -->
   <joint name="wheel_left_joint" type="continuous">
-    <parent link="base_link"/>
-    <child link="left_wheel"/>
+    <parent link="shelfino2/base_link"/>
+    <child link="shelfino2/left_wheel"/>
     <origin xyz="0 0.27 0.125" rpy="0 1.5707 1.5707"/>
     <axis xyz="0 0 1"/>
@@ -57,5 +57,5 @@
                                                       LEFT WHEEL
 -->
-  <link name="left_wheel">
+  <link name="shelfino2/left_wheel">
     <visual name="visual">
       <geometry>
@@ -80,6 +80,6 @@
 -->
   <joint name="wheel_right_joint" type="continuous">
-    <parent link="base_link"/>
-    <child link="right_wheel"/>
+    <parent link="shelfino2/base_link"/>
+    <child link="shelfino2/right_wheel"/>
     <origin xyz="0 -0.27 0.125" rpy="0 1.5707 1.5707"/>
     <axis xyz="0 0 1"/>
@@ -88,5 +88,5 @@
                                                       RIGHT WHEEL
 -->
-  <link name="right_wheel">
+  <link name="shelfino2/right_wheel">
     <visual name="visual">
       <geometry>
@@ -111,6 +111,6 @@
 -->
   <joint name="lidar2d_joint" type="fixed">
-    <parent link="base_link"></parent>
-    <child link="base_laser"></child>
+    <parent link="shelfino2/base_link"></parent>
+    <child link="shelfino2/base_laser"></child>
     <origin xyz="0 0 0.45" rpy="0 0 0"/>
   </joint>
@@ -118,5 +118,5 @@
                                                       LIDAR
 -->
-  <link name="base_laser">
+  <link name="shelfino2/base_laser">
     <visual>
       <geometry>

Commit message: More multiple robot fixes

File: shelfino_description/models/shelfino/model.xacro (robot description, xacro)
@@ -1,141 +1,145 @@
 <?xml version='1.0'?>
-<robot name="shelfino">
-<!--
-                                                      MATERIALS
--->
-  <material name="black">
-      <color rgba="0.1 0.1 0.1 1.0"/>
-  </material>
-  <material name="grey">
-    <color rgba="0.7 0.7 0.7 1.0"/>
-  </material>
-  <material name="white">
-    <color rgba="1.0 1.0 1.0 1.0"/>
-  </material>
-<!--
-                                                      BODY OF SHELFINO
--->
-  <link name='shelfino2/base_link'>
-    <visual name='body_visual'>
-      <origin xyz='0 0 .25'/>
-      <geometry>
-        <box size=".5 .5 .4" />
-      </geometry>
-      <material name="grey" />
-    </visual>
-    <visual name='front_caster_visual'>
-      <origin xyz='-0.2 0 0.05'/>
-      <geometry>
-        <sphere radius=".05" />
-      </geometry>
-      <material name="white" />
-    </visual>
-    <visual name='back_caster_visual'>
-      <origin xyz='0.2 0 0.05'/>
-      <geometry>
-        <sphere radius=".05" />
-      </geometry>
-      <material name="white" />
-    </visual>
-    <collision name='collision'>
-      <origin xyz='0 0 .225'/>
-      <geometry>
-        <box size=".5 .5 .45" />
-      </geometry>
-    </collision>
-  </link>
-<!--
-                                                      LEFT WHEEL JOINT
--->
-  <joint name="wheel_left_joint" type="continuous">
-    <parent link="shelfino2/base_link"/>
-    <child link="shelfino2/left_wheel"/>
-    <origin xyz="0 0.27 0.125" rpy="0 1.5707 1.5707"/>
-    <axis xyz="0 0 1"/>
-  </joint>
-<!--
-                                                      LEFT WHEEL
--->
-  <link name="shelfino2/left_wheel">
-    <visual name="visual">
-      <geometry>
-       <cylinder radius="0.125" length="0.03" />
-      </geometry>
-      <material name="black" />
-    </visual>
-    <collision name="collision">
-      <geometry>
+<robot name="shelfino" xmlns:xacro="http://www.ros.org/wiki/xacro">
+  <xacro:arg name="robot_name" default="shelfinoX" />
+  <xacro:macro name="shelfino" params="robot_name">
+  <!--
+                                                        MATERIALS
+  -->
+    <material name="black">
+        <color rgba="0.1 0.1 0.1 1.0"/>
+    </material>
+    <material name="grey">
+      <color rgba="0.7 0.7 0.7 1.0"/>
+    </material>
+    <material name="white">
+      <color rgba="1.0 1.0 1.0 1.0"/>
+    </material>
+  <!--
+                                                        BODY OF SHELFINO
+  -->
+    <link name='${robot_name}/base_link'>
+      <visual name='body_visual'>
+        <origin xyz='0 0 .25'/>
+        <geometry>
+          <box size=".5 .5 .4" />
+        </geometry>
+        <material name="grey" />
+      </visual>
+      <visual name='front_caster_visual'>
+        <origin xyz='-0.2 0 0.05'/>
+        <geometry>
+          <sphere radius=".05" />
+        </geometry>
+        <material name="white" />
+      </visual>
+      <visual name='back_caster_visual'>
+        <origin xyz='0.2 0 0.05'/>
+        <geometry>
+          <sphere radius=".05" />
+        </geometry>
+        <material name="white" />
+      </visual>
+      <collision name='collision'>
+        <origin xyz='0 0 .225'/>
+        <geometry>
+          <box size=".5 .5 .45" />
+        </geometry>
+      </collision>
+    </link>
+  <!--
+                                                        LEFT WHEEL JOINT
+  -->
+    <joint name="wheel_left_joint" type="continuous">
+      <parent link="${robot_name}/base_link"/>
+      <child link="${robot_name}/left_wheel"/>
+      <origin xyz="0 0.27 0.125" rpy="0 1.5707 1.5707"/>
+      <axis xyz="0 0 1"/>
+    </joint>
+  <!--
+                                                        LEFT WHEEL
+  -->
+    <link name="${robot_name}/left_wheel">
+      <visual name="visual">
+        <geometry>
         <cylinder radius="0.125" length="0.03" />
-      </geometry>
-    </collision>
-    <inertial>
-      <mass value="2.8498940e-02" />
-      <inertia ixx="1.1175580e-05" ixy="-4.2369783e-11" ixz="-5.9381719e-09"
-               iyy="1.1192413e-05" iyz="-1.4400107e-11"
-               izz="2.0712558e-05" />
-    </inertial>
-  </link>
-<!--
-                                                      RIGHT WHEEL JOINT
--->
-  <joint name="wheel_right_joint" type="continuous">
-    <parent link="shelfino2/base_link"/>
-    <child link="shelfino2/right_wheel"/>
-    <origin xyz="0 -0.27 0.125" rpy="0 1.5707 1.5707"/>
-    <axis xyz="0 0 1"/>
-  </joint>
-<!--
-                                                      RIGHT WHEEL
--->
-  <link name="shelfino2/right_wheel">
-    <visual name="visual">
-      <geometry>
-        <cylinder radius="0.125" length="0.03" />
-      </geometry>
-      <material name="black" />
-    </visual>
-    <collision name="collision">
-      <geometry>
-        <cylinder radius="0.125" length="0.03" />
-      </geometry>
-    </collision>
-    <inertial>
-      <mass value="2.8498940e-02" />
-      <inertia ixx="1.1175580e-05" ixy="-4.2369783e-11" ixz="-5.9381719e-09"
-               iyy="1.1192413e-05" iyz="-1.4400107e-11"
-               izz="2.0712558e-05" />
-    </inertial>
-  </link>
-<!--
-                                                      LIDAR FIXED JOINT
--->
-  <joint name="lidar2d_joint" type="fixed">
-    <parent link="shelfino2/base_link"></parent>
-    <child link="shelfino2/base_laser"></child>
-    <origin xyz="0 0 0.45" rpy="0 0 0"/>
-  </joint>
-<!--
-                                                      LIDAR
--->
-  <link name="shelfino2/base_laser">
-    <visual>
-      <geometry>
-        <mesh filename="package://shelfino_gazebo/models/lidar2d/meshes/hokuyo.dae" />
-      </geometry>
-      <material name="black"/>
-    </visual>
-    <collision>
-      <origin xyz="0 0 0.02"/>
-      <geometry>
-        <cylinder length="0.04" radius="0.023"/>
-      </geometry>
-    </collision>
-    <inertial>
-      <mass value="0.1" />
-      <origin xyz="0 0 0" />
-      <inertia ixx="0.001" ixy="0.0" ixz="0.0"
-               iyy="0.001" iyz="0.0"
-               izz="0.001" />
-    </inertial>
-  </link>
+        </geometry>
+        <material name="black" />
+      </visual>
+      <collision name="collision">
+        <geometry>
+          <cylinder radius="0.125" length="0.03" />
+        </geometry>
+      </collision>
+      <inertial>
+        <mass value="2.8498940e-02" />
+        <inertia ixx="1.1175580e-05" ixy="-4.2369783e-11" ixz="-5.9381719e-09"
+                iyy="1.1192413e-05" iyz="-1.4400107e-11"
+                izz="2.0712558e-05" />
+      </inertial>
+    </link>
+  <!--
+                                                        RIGHT WHEEL JOINT
+  -->
+    <joint name="wheel_right_joint" type="continuous">
+      <parent link="${robot_name}/base_link"/>
+      <child link="${robot_name}/right_wheel"/>
+      <origin xyz="0 -0.27 0.125" rpy="0 1.5707 1.5707"/>
+      <axis xyz="0 0 1"/>
+    </joint>
+  <!--
+                                                        RIGHT WHEEL
+  -->
+    <link name="${robot_name}/right_wheel">
+      <visual name="visual">
+        <geometry>
+          <cylinder radius="0.125" length="0.03" />
+        </geometry>
+        <material name="black" />
+      </visual>
+      <collision name="collision">
+        <geometry>
+          <cylinder radius="0.125" length="0.03" />
+        </geometry>
+      </collision>
+      <inertial>
+        <mass value="2.8498940e-02" />
+        <inertia ixx="1.1175580e-05" ixy="-4.2369783e-11" ixz="-5.9381719e-09"
+                iyy="1.1192413e-05" iyz="-1.4400107e-11"
+                izz="2.0712558e-05" />
+      </inertial>
+    </link>
+  <!--
+                                                        LIDAR FIXED JOINT
+  -->
+    <joint name="lidar2d_joint" type="fixed">
+      <parent link="${robot_name}/base_link"></parent>
+      <child link="${robot_name}/base_laser"></child>
+      <origin xyz="0 0 0.45" rpy="0 0 0"/>
+    </joint>
+  <!--
+                                                        LIDAR
+  -->
+    <link name="${robot_name}/base_laser">
+      <visual>
+        <geometry>
+          <mesh filename="package://shelfino_gazebo/models/lidar2d/meshes/hokuyo.dae" />
+        </geometry>
+        <material name="black"/>
+      </visual>
+      <collision>
+        <origin xyz="0 0 0.02"/>
+        <geometry>
+          <cylinder length="0.04" radius="0.023"/>
+        </geometry>
+      </collision>
+      <inertial>
+        <mass value="0.1" />
+        <origin xyz="0 0 0" />
+        <inertia ixx="0.001" ixy="0.0" ixz="0.0"
+                iyy="0.001" iyz="0.0"
+                izz="0.001" />
+      </inertial>
+    </link>
+  </xacro:macro>
+  <xacro:shelfino robot_name="$(arg robot_name)" />
 </robot>

Commit message: Multiple robots fixes

File: shelfino_description/models/shelfino/model.xacro (robot description, xacro)
@@ -123,5 +123,5 @@
       <visual>
         <geometry>
-          <mesh filename="package://shelfino_gazebo/models/lidar2d/meshes/hokuyo.dae" />
+          <mesh filename="package://shelfino_description/models/lidar2d/meshes/hokuyo.dae" />
         </geometry>
         <material name="black"/>

Commit message: more strange behaviours being solved.....

File: shelfino_description/models/shelfino/model.xacro (robot description, xacro)
@@ -20,7 +20,7 @@
     <link name='${robot_name}/base_link'>
       <visual name='body_visual'>
-        <origin xyz='0 0 .25'/>
+        <origin xyz='0 0 0.25'/>
         <geometry>
-          <box size=".5 .5 .4" />
+          <box size="0.5 0.5 0.4" />
         </geometry>
         <material name="grey" />
@@ -29,5 +29,5 @@
         <origin xyz='-0.2 0 0.05'/>
         <geometry>
-          <sphere radius=".05" />
+          <sphere radius="0.05" />
         </geometry>
         <material name="white" />
@@ -36,12 +36,12 @@
         <origin xyz='0.2 0 0.05'/>
         <geometry>
-          <sphere radius=".05" />
+          <sphere radius="0.05" />
         </geometry>
         <material name="white" />
       </visual>
       <collision name='collision'>
-        <origin xyz='0 0 .225'/>
+        <origin xyz='0 0 0.225'/>
         <geometry>
-          <box size=".5 .5 .45" />
+          <box size="0.5 0.5 0.45" />
         </geometry>
       </collision>
