Commit message: course modifications

File: shelfino_description/models/shelfino/model.urdf (robot description, URDF)
Before this commit: robot shelfino, 4 links, 3 joints
Links:
- link base_link: geometry collision box size=.5 .5 .45; visual box size=.5 .5 .4

Commit message: organizing

File: shelfino_description/models/shelfino/model.urdf (robot description, URDF)
Before this commit: robot shelfino, 4 links, 3 joints
Links:
- link base_laser: geometry collision cylinder length=0.04 radius=0.023; visual mesh filename=package://shelfino_description/models/lidar2d/meshes/hokuyo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
- link base_link: geometry collision box size=0.5 0.5 0.45; visual box size=0.5 0.5 0.4
