Commit message: multi robot simulation first commit

File: shelfino_description/models/shelfino/model.sdf.xacro (robot description, xacro)
@@ -1,8 +1,10 @@
 <?xml version='1.0'?>
-<sdf version='1.4'>
+<sdf version='1.4' xmlns:xacro="http://www.ros.org/wiki/xacro">
+  <xacro:arg name="robot_name" default="shelfinoX" />
+  <xacro:macro name="shelfino" params="robot_name">
 <!--
                                                       SHELFINO MODEL
 -->
-  <model name="shelfino">
+  <model name="${robot_name}">
 <!--
                                                       BODY OF SHELFINO
@@ -175,5 +177,5 @@
       <ros>
         <!-- Set namespace -->
-        <!-- <namespace>gazebo</namespace> -->
+        <!-- <namespace>${robot_name}</namespace> -->
       </ros>
       <!-- <alwaysOn>true</alwaysOn> -->
@@ -194,6 +196,6 @@
       <publish_odom_tf>true</publish_odom_tf>
       <publish_wheel_tf>false</publish_wheel_tf>
-      <odometry_frame>gazebo/odom</odometry_frame>
-      <robot_base_frame>gazebo/base_link</robot_base_frame>
+      <odometry_frame>${robot_name}/odom</odometry_frame>
+      <robot_base_frame>${robot_name}/base_link</robot_base_frame>
       <!-- <odometrySource>ENCODER</odometrySource> -->
       <!-- <odometrySource>WORLD</odometrySource> -->
@@ -204,5 +206,5 @@
     <plugin name="joint_state" filename="libgazebo_ros_joint_state_publisher.so">
       <ros>
-        <namespace>gazebo</namespace>
+        <namespace>${robot_name}</namespace>
         <remapping>~/out:=joint_states</remapping>
       </ros>
@@ -212,3 +214,5 @@
     </plugin>
   </model>
+  </xacro:macro>
+  <xacro:shelfino robot_name="$(arg robot_name)" />
 </sdf>

Commit message: adding multirobot and added obstacles msg type

File: shelfino_description/models/shelfino/model.sdf.xacro (robot description, xacro)
@@ -161,5 +161,5 @@
     <joint name="lidar2d_joint" type="fixed">
       <parent>base_link</parent>
-      <child>lidar2d::lidar_link</child>
+      <child>lidar_link</child>
       <pose>0 0 0 0 0 0</pose>
     </joint>
@@ -167,8 +167,69 @@
                                                       LIDAR
 -->
-    <include>
-      <uri>model://lidar2d</uri>
+    <link name="lidar_link">
       <pose>0 0 0.45 0 0 0</pose>
-    </include>
+      <inertial>
+        <mass>0.1</mass>
+      </inertial>
+      <visual name="visual">
+        <geometry>
+          <mesh>
+            <uri>model://lidar2d/meshes/hokuyo.dae</uri>
+          </mesh>
+        </geometry>
+      </visual>
+      <collision name="collision-base">
+        <pose>0 0 -0.0145 0 0 0</pose>
+        <geometry>
+          <box>
+            <size>0.05 0.05 0.041</size>
+          </box>
+        </geometry>
+      </collision>
+      <collision name="collision-top">
+        <pose>0 0 0.0205 0 0 0</pose>
+        <geometry>
+          <cylinder>
+            <radius>0.021</radius>
+            <length>0.029</length>
+          </cylinder>
+        </geometry>
+      </collision>
+      <sensor name="laser" type="ray">
+        <always_on>true</always_on>
+        <visualize>false</visualize>
+        <update_rate>30</update_rate>
+        <pose>0 0 0.03 0 0 0</pose>
+        <ray>
+          <scan>
+            <horizontal>
+              <samples>360</samples>
+              <resolution>1</resolution>
+              <min_angle>0</min_angle>
+              <max_angle>6.28318530718</max_angle>
+            </horizontal>
+          </scan>
+          <range>
+            <min>0.15</min>
+            <max>12.</max>
+            <resolution>0.01</resolution>
+          </range>
+          <noise>
+            <type>gaussian</type>
+            <mean>0.0</mean>
+            <stddev>0.02</stddev>
+          </noise>
+        </ray>
+        <plugin name="laser" filename="libgazebo_ros_ray_sensor.so">
+          <ros>
+            <!-- Set namespace -->
+            <namespace>${robot_name}</namespace>
+            <remapping>~/out:=scan</remapping>
+          </ros>
+          <output_type>sensor_msgs/LaserScan</output_type>
+          <frame_name>${robot_name}/base_laser</frame_name>
+        </plugin>
+      </sensor>
+    </link>
 <!--
                                                       DIFFERENTIAL DRIVE CONTROLLER
@@ -177,5 +238,5 @@
       <ros>
         <!-- Set namespace -->
-        <!-- <namespace>${robot_name}</namespace> -->
+        <namespace>${robot_name}</namespace>
       </ros>
       <!-- <alwaysOn>true</alwaysOn> -->
@@ -191,5 +252,5 @@
       <max_wheel_torque>20</max_wheel_torque>
       <max_wheel_acceleration>1.0</max_wheel_acceleration>
-      <command_topic>cmd_vel</command_topic>
+      <command_topic>${robot_name}/cmd_vel</command_topic>
       <!-- output -->
       <publish_odom>true</publish_odom>
